File: MoteinoLeo/Moteino_Leo.brd (EAGLE design)
At the start: 35.8 x 23.1 mm, 22 parts, among them IC3 MCP1703CB, U3 ATMEGA32U4, X1 16Mhz

Commit message: Update to R1 production board
Parts:
- added F1: PTC0805, LowPowerLab:0805-PTC
- moved R4 3.72 mm to (6.86, 8.74), turned to 270 degrees
- moved U$1 2.54 mm to (32.3, 18.3)
- moved R3 1.80 mm to (8.76, 8.74), turned to 270 degrees
- moved R1 0.89 mm to (10.0, 17.8)
- moved C5 0.88 mm to (14.4, 17.5), turned to 270 degrees
- moved C1 0.13 mm to (11.2, 8.51)
- moved C2 0.13 mm to (12.7, 15.5)
- turned R2 to 0 degrees
- turned U$2 to 0 degrees
Connections:
- removed net N$2: R2.1, U$2.PLUS
- new net N$1: R2.2, U$2.MINUS
- new net USBPOWER: F1.2, JP3.VBUS
- net D13: now also U$2.PLUS
- net GND: now also R2.1; no longer U$2.MINUS
- net TXO: no longer R2.2
- net VBUS: now also F1.1; no longer JP3.VBUS
Routing:
- net TXO: track 10.7 -> 0.00 mm
- net GND: track 113.9 -> 107.2 mm, vias 5 -> 14
- net D+: track 3.35 -> 9.04 mm
- net D13: track 20.3 -> 24.7 mm
- net N$8: track 6.74 -> 10.7 mm
- net D-: track 2.84 -> 6.25 mm
- net USBPOWER: track 0.00 -> 2.95 mm
- net VBUS: track 28.2 -> 25.3 mm
- net N$3: track 6.91 -> 4.37 mm
- net N$2: track 2.34 -> 0.00 mm
- net N$1: track 0.00 -> 2.34 mm
- net D12: track 16.7 -> 15.7 mm
- net RST: track 23.8 -> 22.9 mm
- net A3: track 12.7 -> 13.5 mm
- net VCC: track 64.0 -> 64.7 mm
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Other:
- board text removed: "AREF"
