File: R4/Moteino.sch (EAGLE design)
At the start: 20 parts, among them IC3 MCP1703CB, X1 16 MHz

Commit message: Add Moteino R4 & R4-USB
Parts:
- removed U$4: AT25F512BJEDEC, LowPowerLab:AT25F512BJEDEC
- added U$5: RFM69, LowPowerLab:RFM69
- added U$6: AT25F512BWIDE_5.3MM, LowPowerLab:AT25F512BWIDE_5.3MM
Connections:
- net D10_SS: now also U$5.SEL
- net D11_MOSI: now also U$5.MOSI, U$6.SI; no longer U$4.SI
- net D12_MISO: now also U$5.MISO, U$6.SO; no longer U$4.SO
- net D13_SCK: now also U$5.SCK, U$6.SCK; no longer U$4.SCK
- net D2: now also U$5.DIO0
- net D8: now also U$6.CS; no longer U$4.CS
- net GND: now also U$5.GND, U$6.GND; no longer U$4.GND
- net N$3: now also U$5.ANT
- net VCC: now also U$5.VCC, U$6.HOLD, U$6.VCC, U$6.WP; no longer U$4.HOLD, U$4.VCC, U$4.WP
Other:
- note added: "Moteino R4"
- note removed: "Moteino"
- moved on the sheet: C1, FTDI

Commit message: Update Eagle files, add schematic PDFs
Parts:
- renumbered U$6 to W25X40CLSNIG-ND
Other:
- note added: "RFM12B"
- moved on the sheet: +, ANALOGSIDE, ATMEGA328, C5, DIGITALSIDE, JP1, JP2, R1, X1
