File: R4USB/Moteino.sch (EAGLE design)
At the start: 28 parts, among them CN1 MINIB, IC1 FT232RL, IC3 MCP1703CB, X1 16 MHz

Commit message: Update Eagle files, add schematic PDFs
Parts:
- removed U$6: AT25F512BWIDE_5.3MM, LowPowerLab:AT25F512BWIDE_5.3MM
- added W25X40CLSNIG-ND: AT25F512BWIDE_5.3MM, LowPowerLab:AT25F512BWIDE_5.3MM
Connections:
- net D11_MOSI: now also W25X40CLSNIG-ND.SI; no longer U$6.SI
- net D12_MISO: now also W25X40CLSNIG-ND.SO; no longer U$6.SO
- net D13_SCK: now also W25X40CLSNIG-ND.SCK; no longer U$6.SCK
- net D8: now also W25X40CLSNIG-ND.CS; no longer U$6.CS
- net GND: now also W25X40CLSNIG-ND.GND; no longer U$6.GND
- net VCC: now also W25X40CLSNIG-ND.HOLD, W25X40CLSNIG-ND.VCC, W25X40CLSNIG-ND.WP; no longer U$6.HOLD, U$6.VCC, U$6.WP
Other:
- note added: "Moteino R4-USB"
- note added: "RFM12B"
- note removed: "Moteino R4"
- moved on the sheet: +, ANALOGSIDE, ATMEGA328, C1, C5, C6, CN1, DIGITALSIDE, IC1, JP1, JP2, R1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
